File: fml13v01-uart-ec.kicad_pcb (KiCad board)
At the start: 2 copper layers, 26 x 30 mm, 10 parts, among them J1 Conn_01x03, J3 Conn_01x03_Pin, P1 USB_C_Plug

Commit message: Corrected Rx/Tx lines on JST connector for RPi Dbg UART
Parts:
- J1: value Conn_01x03 -> JST_UART
- J3: value Conn_01x03_Pin -> PinHeader_UART
Connections:
- J3 pad 1: Net-(J1-Pin_1) -> Net-(J1-Pin_3)
- J3 pad 2: Net-(J1-Pin_3) -> Net-(J1-Pin_1)
- P1 pad A8: Net-(J1-Pin_1) -> Net-(J1-Pin_3)
- P1 pad B8: Net-(J1-Pin_3) -> Net-(J1-Pin_1)
Routing:
- net Net-(J1-Pin_3): track 34.2 -> 29.4 mm
Changed lines of the file:
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@@
 			(size 0.38 1)
 			(layers "F.Cu" "F.Mask" "F.Paste")
-			(net 3 "Net-(J1-Pin_1)")
+			(net 2 "Net-(J1-Pin_3)")
 			(pinfunction "SBU1")
 			(pintype "bidirectional")
@@
 			(size 0.38 1)
 			(layers "B.Cu" "B.Mask" "B.Paste")
-			(net 2 "Net-(J1-Pin_3)")
+			(net 3 "Net-(J1-Pin_1)")
 			(pinfunction "SBU2")
 			(pintype "bidirectional")
@@
 			)
 		)
-		(property "Value" "Conn_01x03_Pin"
+		(property "Value" "PinHeader_UART"
 			(at 4.385 7.35 90)
 			(layer "F.Fab")
@@
 			(layers "*.Cu" "*.Mask")
 			(remove_unused_layers no)
-			(net 3 "Net-(J1-Pin_1)")
+			(net 2 "Net-(J1-Pin_3)")
 			(pinfunction "Pin_1")
 			(pintype "passive")
@@
 			(layers "*.Cu" "*.Mask")
 			(remove_unused_layers no)
-			(net 2 "Net-(J1-Pin_3)")
+			(net 3 "Net-(J1-Pin_1)")
 			(pinfunction "Pin_2")
 			(pintype "passive")
@@
 			)
 		)
-		(property "Value" "Conn_01x03"
+		(property "Value" "JST_UART"
 			(at 0 3.98 0)
 			(layer "F.Fab")
@@
 	)
 	(segment
-		(start 143 154)
-		(end 146 154)
+		(start 139.025 140.975)
+		(end 139.025 146.125)
 		(width 0.1524)
 		(layer "F.Cu")
@@
 	)
 	(segment
-		(start 147 153)
+		(start 143.125 146.125)
+		(end 147 150)
+		(width 0.1524)
+		(layer "F.Cu")
+		(net 2)
+	)
+	(segment
+		(start 140.75 139.25)
+		(end 139.025 140.975)
+		(width 0.1524)
+		(layer "F.Cu")
+		(net 2)
+	)
+	(segment
+		(start 147 150)
 		(end 147 152)
 		(width 0.1524)
@@
 	)
 	(segment
-		(start 146 154)
-		(end 147 153)
+		(start 139.025 146.125)
+		(end 143.125 146.125)
 		(width 0.1524)
 		(layer "F.Cu")
@@
 	)
 	(segment
-		(start 136.485 146.125)
-		(end 136.485 147.485)
+		(start 140.75 129.04)
+		(end 140.75 139.25)
 		(width 0.1524)
 		(layer "F.Cu")
@@
 	)
 	(segment
-		(start 136.485 147.485)
-		(end 143 154)
+		(start 136.485 146.125)
+		(end 138.86 148.5)
 		(width 0.1524)
 		(layer "F.Cu")
-		(net 2)
+		(net 3)
+	)
+	(segment
+		(start 145 150.5)
+		(end 145 152)
+		(width 0.1524)
+		(layer "F.Cu")
+		(net 3)
+	)
+	(segment
+		(start 143 148.5)
+		(end 145 150.5)
+		(width 0.1524)
+		(layer "F.Cu")
+		(net 3)
+	)
+	(segment
+		(start 138.86 148.5)
+		(end 143 148.5)
+		(width 0.1524)
+		(layer "F.Cu")
+		(net 3)
 	)
 	(segment
@@
 		(width 0.1524)
 		(layer "B.Cu")
-		(net 2)
+		(net 3)
 	)
 	(segment
@@
 		(width 0.1524)
 		(layer "B.Cu")
-		(net 2)
+		(net 3)
 	)
 	(segment
@@
 		(width 0.1524)
 		(layer "B.Cu")
-		(net 2)
-	)
-	(segment
-		(start 139.025 140.975)
-		(end 139.025 146.125)
-		(width 0.1524)
-		(layer "F.Cu")
 		(net 3)
 	)
-	(segment
-		(start 143.5 153.5)
-		(end 144.5 153.5)
-		(width 0.1524)
-		(layer "F.Cu")
-		(net 3)
-	)
-	(segment
-		(start 139.025 149.025)
-		(end 143.5 153.5)
-		(width 0.1524)
-		(layer "F.Cu")
-		(net 3)
-	)
-	(segment
-		(start 145 153)
-		(end 145 152)
-		(width 0.1524)
-		(layer "F.Cu")
-		(net 3)
-	)
-	(segment
-		(start 144.5 153.5)
-		(end 145 153)
-		(width 0.1524)
-		(layer "F.Cu")
-		(net 3)
-	)
-	(segment
-		(start 140.75 139.25)
-		(end 139.025 140.975)
-		(width 0.1524)
-		(layer "F.Cu")
-		(net 3)
-	)
-	(segment
-		(start 139.025 146.125)
-		(end 139.025 149.025)
-		(width 0.1524)
-		(layer "F.Cu")
-		(net 3)
-	)
-	(segment
-		(start 140.75 129.04)
-		(end 140.75 139.25)
-		(width 0.1524)
-		(layer "F.Cu")
-		(net 3)
-	)
